File: HW Design/Main Board/KiCAD Files/OpenSystem-Drone.kicad_pcb (KiCad board)
At the start: 2 copper layers, 14 parts, among them J1 Conn_01x02_Female, J2 CAN_2, J3 CAN_1, J4 CAN_2, J5 CAN_1, U1 LM3940IMP-3.3/NOPB, U2 SN65HVD232, U3 SN65HVD232, U4 SN65HVD232, U5 STM32F446ZETx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

Commit message: hw desgign updates
Parts:
- removed J4: CAN_2, Connector_Wuerth:Wuerth_WR-WTB_64800411622_1x04_P1.50mm_Vertical
- removed U3: SN65HVD232, Package_SO:SOIC-8_3.9x4.9mm_P1.27mm
- removed U6: STM32F103RET6, Package_QFP:LQFP-64_10x10mm_P0.5mm
- added C1: 0.47 uF, Capacitor_SMD:C_1206_3216Metric, F.Cu at (25.9, 82.0)
- added C2: 33uF, Capacitor_SMD:C_1206_3216Metric, F.Cu at (31.6, 82.0)
- added C3: 100nF, Capacitor_SMD:C_1206_3216Metric, F.Cu at (118.9, 128.5)
- added C4: 1uF, Capacitor_SMD:C_1206_3216Metric, F.Cu at (113.2, 128.5)
- added C5: 100uF, Capacitor_SMD:C_1206_3216Metric, F.Cu at (37.1, 95.0)
- added C6: 10uF, Capacitor_SMD:C_1206_3216Metric, F.Cu at (31.4, 98.3)
- added C7: C, Capacitor_SMD:C_1206_3216Metric, F.Cu at (31.4, 101.7)
- added C8: C, Capacitor_SMD:C_1206_3216Metric, F.Cu at (31.4, 95.0)
- added J6: CAN_1, Connector_Wuerth:Wuerth_WR-WTB_64800411622_1x04_P1.50mm_Vertical, F.Cu at (235.5, 81.3)
- added JP1: SolderJumper_3_Bridged12, Jumper:SolderJumper-3_P1.3mm_Open_Pad1.0x1.5mm_NumberLabels, F.Cu at (26.5, 134.5)
- added JP2: SolderJumper_3_Bridged12, Jumper:SolderJumper-3_P1.3mm_Open_Pad1.0x1.5mm_NumberLabels, F.Cu at (26.5, 130.9)
- added R1: 0, Resistor_SMD:R_1206_3216Metric, F.Cu at (46.3, 82.0)
- added R2: 0, Resistor_SMD:R_1206_3216Metric, F.Cu at (40.7, 82.0)
- added R3: R, Resistor_SMD:R_1206_3216Metric, F.Cu at (37.1, 101.6)
- added R4: 4k7, Resistor_SMD:R_1206_3216Metric, F.Cu at (42.7, 98.3)
- added R5: R, Resistor_SMD:R_1206_3216Metric, F.Cu at (37.1, 98.3)
- added R6: 4k7, Resistor_SMD:R_1206_3216Metric, F.Cu at (42.7, 95.0)
- J2: value CAN_2 -> MicroSD; footprint Connector_Wuerth:Wuerth_WR-WTB_64800411622_1x04_P1.50mm_Vertical -> KiCAD Footprints:MicroSD
- moved J2 152.7 mm to (129.5, 157.5), turned to 0 degrees
- moved U8 87.0 mm to (52.8, 112.0)
- moved U7 77.2 mm to (67.3, 82.5)
Connections:
- J2 pad 1: +5V -> unconnected-(J2-Pad1)
- J2 pad 2: CAN_2_H -> SPI1_SD_CS
- J2 pad 3: CAN_2_L -> SPI1_SD_MOSI
- J2 pad 4: GND -> +3V3
- U5 pad 136: unconnected-(U5-Pad136) -> I2C1_IMU_SCL
- U5 pad 137: unconnected-(U5-Pad137) -> I2C1_IMU_SDA
- U5 pad 40: unconnected-(U5-Pad40) -> SPI1_SD_CS
- U5 pad 41: unconnected-(U5-Pad41) -> SPI1_SD_CLK
- U5 pad 42: unconnected-(U5-Pad42) -> SPI1_SD_MISO
- U5 pad 43: unconnected-(U5-Pad43) -> SPI1_SD_MOSI
- U8 pad 1: unconnected-(U8-Pad1) -> xxx
- U8 pad 10: unconnected-(U8-Pad10) -> IMU_AD2
- U8 pad 11: unconnected-(U8-Pad11) -> +3V3
- U8 pad 12: unconnected-(U8-Pad12) -> xxx
- U8 pad 13: unconnected-(U8-Pad13) -> xxx
- U8 pad 14: unconnected-(U8-Pad14) -> +3V3
- U8 pad 15: unconnected-(U8-Pad15) -> IMU_AD1
- U8 pad 16: unconnected-(U8-Pad16) -> xxx
- U8 pad 3: unconnected-(U8-Pad3) -> +3V3
- U8 pad 4: unconnected-(U8-Pad4) -> GND
- U8 pad 6: unconnected-(U8-Pad6) -> GND
- U8 pad 7: unconnected-(U8-Pad7) -> +3V3
- U8 pad 8: unconnected-(U8-Pad8) -> I2C1_IMU_SCL
- U8 pad 9: unconnected-(U8-Pad9) -> I2C1_IMU_SDA

Commit message: Updates of HW Desgin
Parts:
- removed J6: CAN_1, Connector_Wuerth:Wuerth_WR-WTB_64800411622_1x04_P1.50mm_Vertical
- removed U4: SN65HVD232, Package_SO:SOIC-8_3.9x4.9mm_P1.27mm
- added C10: 4u7, Capacitor_SMD:C_1206_3216Metric, F.Cu at (102.9, 31.8)
- added C11: 100n, Capacitor_SMD:C_1206_3216Metric, F.Cu at (114.2, 31.8)
- added C12: 1u, Capacitor_SMD:C_1206_3216Metric, F.Cu at (102.9, 35.1)
- added C13: 100n, Capacitor_SMD:C_1206_3216Metric, F.Cu at (108.5, 31.8)
- added C14: 10n, Capacitor_SMD:C_1206_3216Metric, F.Cu at (108.5, 35.1)
- added C15: 100n, Capacitor_SMD:C_1206_3216Metric, F.Cu at (114.2, 28.4)
- added C16: 100n, Capacitor_SMD:C_1206_3216Metric, F.Cu at (97.2, 35.1)
- added C17: 100n, Capacitor_SMD:C_1206_3216Metric, F.Cu at (102.9, 38.5)
- added C18: 100n, Capacitor_SMD:C_1206_3216Metric, F.Cu at (108.5, 38.5)
- added C19: 100n, Capacitor_SMD:C_1206_3216Metric, F.Cu at (97.2, 31.8)
- added C20: 100n, Capacitor_SMD:C_1206_3216Metric, F.Cu at (119.8, 28.4)
- added C21: 12p, Capacitor_SMD:C_1206_3216Metric, F.Cu at (226.1, 62.2)
- added C22: 100n, Capacitor_SMD:C_1206_3216Metric, F.Cu at (97.2, 28.4)
- added C23: 100n, Capacitor_SMD:C_1206_3216Metric, F.Cu at (102.9, 28.4)
- added C24: 12p, Capacitor_SMD:C_1206_3216Metric, F.Cu at (219.7, 62.2)
- added C25: 100n, Capacitor_SMD:C_1206_3216Metric, F.Cu at (97.2, 38.5)
- added C26: 100n, Capacitor_SMD:C_1206_3216Metric, F.Cu at (119.8, 31.8)
- added J4: USB C, KiCAD Footprints:usb_c_amphenol, B.Cu at (205.7, 44.5)
- added JP3: SolderJumper_3_Bridged12, Jumper:SolderJumper-3_P1.3mm_Open_Pad1.0x1.5mm_NumberLabels, F.Cu at (97.2, 47.6)
- added JP4: SolderJumper_3_Bridged12, Jumper:SolderJumper-3_P1.3mm_Open_Pad1.0x1.5mm_NumberLabels, F.Cu at (97.2, 51.2)
- added JP5: SolderJumper_3_Bridged12, Jumper:SolderJumper-3_P1.3mm_Open_Pad1.0x1.5mm_NumberLabels, F.Cu at (148.6, 41.9)
- added Q1: AO3401A, Package_TO_SOT_SMD:SOT-23, F.Cu at (128.5, 28.9)
- added R10: 4k7, Resistor_SMD:R_1206_3216Metric, F.Cu at (108.5, 47.5)
- added R12: 4k7, Resistor_SMD:R_1206_3216Metric, F.Cu at (102.8, 47.5)
- added R9: R, Resistor_SMD:R_1206_3216Metric, F.Cu at (102.8, 50.8)
- added U3: BMP581, KiCAD Footprints:BMP581, F.Cu at (160.0, 33.0)
- C5: value 100uF -> 100nF
- C7: value C -> 100nF
- J2, J3, J5: moved to B.Cu
- R3: value R -> 4k7
- U5: value STM32F446ZETx -> STM32F446RETx; footprint Package_QFP:LQFP-144_20x20mm_P0.5mm -> Package_QFP:LQFP-64_10x10mm_P0.5mm
- Y1: value Crystal_GND2 -> 16MHZ
- moved R2 179.3 mm to (218.4, 58.4)
- moved J2 171.9 mm to (259.1, 44.5), turned to -90 degrees
- moved Y1 132.3 mm to (228.6, 52.1)
- moved U5 117.9 mm to (228.6, 36.8)
- moved C3 109.1 mm to (218.4, 83.8)
- moved C4 109.1 mm to (212.8, 83.8)
- moved U2 66.8 mm to (245.1, 55.9), turned to -90 degrees
- moved J5 63.4 mm to (238.1, 66.5), turned to 0 degrees
- moved J3 55.1 mm to (247.4, 66.5), turned to 0 degrees
Connections:
- net IMU_AD1 renamed ACC_AD
- net IMU_AD2 renamed GYR_AD
- JP1 pad 1: Net-(JP1-Pad1) -> GND
- JP1 pad 3: GND -> Net-(R4-Pad2)
- JP2 pad 1: Net-(JP2-Pad1) -> GND
- JP2 pad 3: GND -> Net-(R6-Pad2)
- R2 pad 1: RCC_OSC_OUT -> Net-(R2-Pad1)
- R2 pad 2: Net-(R2-Pad2) -> HSE_OUT
- R3 pad 2: I2C1_IMU_SDA -> Net-(JP5-Pad3)
- R4 pad 1: Net-(JP1-Pad1) -> +3V3
- R4 pad 2: +3V3 -> Net-(R4-Pad2)
- R5 pad 2: I2C1_IMU_SDA -> I2C1_SCL
- R6 pad 1: Net-(JP2-Pad1) -> +3V3
- R6 pad 2: +3V3 -> Net-(R6-Pad2)
- U2 pad 1: F4_CAN1_TX -> CAN1_TX
- U2 pad 4: F4_CAN1_RX -> CAN1_RX
- U5 pad 1: unconnected-(U5-Pad1) -> +3V3
- U5 pad 12: unconnected-(U5-Pad12) -> GND
- U5 pad 13: unconnected-(U5-Pad13) -> +3.3VA
- U5 pad 16: GND -> unconnected-(U5-Pad16)
- U5 pad 18: unconnected-(U5-Pad18) -> GND
- U5 pad 19: unconnected-(U5-Pad19) -> +3V3
- U5 pad 20: unconnected-(U5-Pad20) -> SPI1_SD_CS
- U5 pad 21: unconnected-(U5-Pad21) -> SPI1_SD_CLK
- U5 pad 22: unconnected-(U5-Pad22) -> SPI1_SD_MISO
- U5 pad 23: RCC_OSC_IN -> SPI1_SD_MOSI
- U5 pad 24: RCC_OSC_OUT -> unconnected-(U5-Pad24)
- U5 pad 25: NRST -> unconnected-(U5-Pad25)
- U5 pad 30: unconnected-(U5-Pad30) -> Net-(C4-Pad1)
- U5 pad 32: unconnected-(U5-Pad32) -> +3V3
- U5 pad 38: GND -> unconnected-(U5-Pad38)
- U5 pad 40: SPI1_SD_CS -> unconnected-(U5-Pad40)
- U5 pad 41: SPI1_SD_CLK -> unconnected-(U5-Pad41)
- U5 pad 42: SPI1_SD_MISO -> unconnected-(U5-Pad42)
- U5 pad 43: SPI1_SD_MOSI -> unconnected-(U5-Pad43)
- U5 pad 44: unconnected-(U5-Pad44) -> USB_D-
- U5 pad 45: unconnected-(U5-Pad45) -> USB_D+
- U5 pad 46: unconnected-(U5-Pad46) -> SWDIO
- U5 pad 47: unconnected-(U5-Pad47) -> GND
- U5 pad 48: unconnected-(U5-Pad48) -> +3V3
- U5 pad 49: unconnected-(U5-Pad49) -> SWCLK
- U5 pad 5: unconnected-(U5-Pad5) -> HSE_IN
- U5 pad 51: GND -> unconnected-(U5-Pad51)
- U5 pad 55: unconnected-(U5-Pad55) -> SWO
- U5 pad 58: unconnected-(U5-Pad58) -> I2C1_SCL
- U5 pad 59: unconnected-(U5-Pad59) -> I2C1_SDA
- U5 pad 6: unconnected-(U5-Pad6) -> HSE_OUT
- U5 pad 61: GND -> unconnected-(U5-Pad61)
- U5 pad 63: unconnected-(U5-Pad63) -> GND
- U5 pad 64: unconnected-(U5-Pad64) -> +3V3
- U5 pad 7: unconnected-(U5-Pad7) -> NRST
- U5 pad 8: unconnected-(U5-Pad8) -> CAN1_RX
- U5 pad 9: unconnected-(U5-Pad9) -> CAN1_TX
- U7 pad A1: unconnected-(U7-PadA1) -> +3V3
- U7 pad A3: unconnected-(U7-PadA3) -> I2C1_SCL
- U7 pad A5: unconnected-(U7-PadA5) -> MAG_AD2
- U7 pad B2: unconnected-(U7-PadB2) -> +3V3
- U7 pad B4: unconnected-(U7-PadB4) -> I2C1_SDA
- U7 pad C1: unconnected-(U7-PadC1) -> MAG_AD1
- U7 pad C5: unconnected-(U7-PadC5) -> GND
- U7 pad D2: unconnected-(U7-PadD2) -> INT_MAG
- U7 pad D4: unconnected-(U7-PadD4) -> DRY_MAG
- U7 pad E1: unconnected-(U7-PadE1) -> GND
- U7 pad E3: unconnected-(U7-PadE3) -> GND
- U7 pad E5: unconnected-(U7-PadE5) -> +3V3
- U8 pad 8: I2C1_IMU_SCL -> I2C1_SCL
- U8 pad 9: I2C1_IMU_SDA -> I2C1_SDA
- Y1 pad 1: Net-(R2-Pad2) -> HSE_IN
- Y1 pad 3: Net-(R1-Pad2) -> Net-(R2-Pad1)
