File: HW Design/Main Board/KiCAD Files/OpenSystem-Drone.kicad_sch (KiCad schematic)
At the start: 0 parts

Commit message: hw desgign updates
Other:
- removed sheet MCU F1

Commit message: Updates of HW Desgin
Other:
- added sheet Internal Communication (internal_comm.kicad_sch)
- added sheet Internal Sensors 2 (internal_sensors_2.kicad_sch)
