File: HW Design/Main Board/KiCAD Files/external_communication.kicad_sch (KiCad schematic)
At the start: 8 parts, among them J2 CAN_2, J3 CAN_1, J4 CAN_2, J5 CAN_1, J6 CAN_1, U2 SN65HVD232, U3 SN65HVD232, U4 SN65HVD232

Commit message: hw desgign updates
Parts:
- removed J2, J4: CAN_2, Connector_Wuerth:Wuerth_WR-WTB_64800411622_1x04_P1.50mm_Vertical, symbol Connector:Conn_01x04_Female
- removed U3: SN65HVD232, Package_SO:SOIC-8_3.9x4.9mm_P1.27mm, symbol Interface_CAN_LIN:SN65HVD232
Connections:
- net F4_CAN1_RX is gone; now on net CAN1_RX: U2.4 (R)
- net F4_CAN1_TX is gone; now on net CAN1_TX: U2.1 (D)
- net F1_CAN1_RX renamed CAN1_RX
- net F1_CAN1_TX renamed CAN1_TX
Other:
- note removed: "CAN_2 BUS"

Commit message: Updates of HW Desgin
Parts:
- removed J6: CAN_1, Connector_Wuerth:Wuerth_WR-WTB_64800411622_1x04_P1.50mm_Vertical, symbol Connector:Conn_01x04_Female
- removed U4: SN65HVD232, Package_SO:SOIC-8_3.9x4.9mm_P1.27mm, symbol Interface_CAN_LIN:SN65HVD232
