File: HW Design/Main Board/KiCAD Files/external_connectors.kicad_sch (KiCad schematic)
At the start: 1 part, among them J1 Conn_01x02_Female

Commit message: hw desgign updates
Parts:
- added J2: MicroSD, KiCAD Footprints:MicroSD, symbol MicroSD:5033981892
Connections:
- net GND: now also J2.11 (CASE), J2.12 (CASE), J2.13 (CASE), J2.14 (CASE), J2.6 (VSS)
- new net +3V3: J2.4 (VDD)
- new net SPI1_SD_CLK: J2.5 (CLK)
- new net SPI1_SD_CS: J2.2 (CD/DAT3)
- new net SPI1_SD_MISO: J2.7 (DAT0)
- new net SPI1_SD_MOSI: J2.3 (CMD)
Other:
- note added: "MicroSD Card Slot"
Changed lines of the file:
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@@
 (kicad_sch (version 20211123) (generator eeschema)
   (paper "A4")
+  (junction (at 182.245 59.69) (diameter 0) (color 0 0 0 0)
+  )
+  (junction (at 153.035 59.69) (diameter 0) (color 0 0 0 0)
+  )
+  (junction (at 159.385 59.69) (diameter 0) (color 0 0 0 0)
+  )
+  (junction (at 146.685 59.69) (diameter 0) (color 0 0 0 0)
+  )
+  (wire (pts (xy 113.03 23.495) (xy 113.03 31.115))
+    (stroke (width 0) (type default) (color 0 0 0 0))
+  )
+  (wire (pts (xy 116.205 36.195) (xy 83.82 36.195))
+    (stroke (width 0) (type default) (color 0 0 0 0))
+  )
+  (wire (pts (xy 146.685 56.515) (xy 146.685 59.69))
+    (stroke (width 0) (type default) (color 0 0 0 0))
+  )
+  (wire (pts (xy 182.245 38.735) (xy 182.245 59.69))
+    (stroke (width 0) (type default) (color 0 0 0 0))
+  )
   (wire (pts (xy 43.815 42.545) (xy 49.53 42.545))
     (stroke (width 0) (type default) (color 0 0 0 0))
   )
+  (wire (pts (xy 105.41 28.575) (xy 107.95 28.575))
+    (stroke (width 0) (type default) (color 0 0 0 0))
+  )
   (wire (pts (xy 49.53 42.545) (xy 49.53 45.085))
     (stroke (width 0) (type default) (color 0 0 0 0))
   )
+  (wire (pts (xy 141.605 59.69) (xy 146.685 59.69))
+    (stroke (width 0) (type default) (color 0 0 0 0))
+  )
+  (wire (pts (xy 182.245 36.195) (xy 192.405 36.195))
+    (stroke (width 0) (type default) (color 0 0 0 0))
+  )
+  (polyline (pts (xy 71.12 72.39) (xy 212.09 72.39))
+    (stroke (width 0) (type default) (color 0 0 0 0))
+  )
+  (wire (pts (xy 83.82 36.195) (xy 83.82 33.655))
+    (stroke (width 0) (type default) (color 0 0 0 0))
+  )
+  (wire (pts (xy 105.41 38.735) (xy 116.205 38.735))
+    (stroke (width 0) (type default) (color 0 0 0 0))
+  )
+  (wire (pts (xy 113.03 31.115) (xy 116.205 31.115))
+    (stroke (width 0) (type default) (color 0 0 0 0))
+  )
+  (wire (pts (xy 159.385 56.515) (xy 159.385 59.69))
+    (stroke (width 0) (type default) (color 0 0 0 0))
+  )
+  (wire (pts (xy 159.385 59.69) (xy 182.245 59.69))
+    (stroke (width 0) (type default) (color 0 0 0 0))
+  )
+  (wire (pts (xy 146.685 59.69) (xy 153.035 59.69))
+    (stroke (width 0) (type default) (color 0 0 0 0))
+  )
+  (wire (pts (xy 107.95 33.655) (xy 116.205 33.655))
+    (stroke (width 0) (type default) (color 0 0 0 0))
+  )
+  (wire (pts (xy 153.035 59.69) (xy 159.385 59.69))
+    (stroke (width 0) (type default) (color 0 0 0 0))
+  )
+  (wire (pts (xy 141.605 56.515) (xy 141.605 59.69))
+    (stroke (width 0) (type default) (color 0 0 0 0))
+  )
   (wire (pts (xy 49.53 37.465) (xy 49.53 40.005))
     (stroke (width 0) (type default) (color 0 0 0 0))
   )
-  (polyline (pts (xy 31.115 55.245) (xy 74.295 55.245))
-    (stroke (width 0) (type default) (color 0 0 0 0))
-  )
-  (polyline (pts (xy 74.295 27.305) (xy 74.295 55.245))
+  (wire (pts (xy 107.95 28.575) (xy 107.95 33.655))
+    (stroke (width 0) (type default) (color 0 0 0 0))
+  )
+  (polyline (pts (xy 27.305 72.39) (xy 71.12 72.39))
+    (stroke (width 0) (type default) (color 0 0 0 0))
+  )
+  (wire (pts (xy 153.035 56.515) (xy 153.035 59.69))
+    (stroke (width 0) (type default) (color 0 0 0 0))
+  )
+  (wire (pts (xy 182.245 59.69) (xy 182.245 62.23))
+    (stroke (width 0) (type default) (color 0 0 0 0))
+  )
+  (wire (pts (xy 105.41 23.495) (xy 113.03 23.495))
+    (stroke (width 0) (type default) (color 0 0 0 0))
+  )
+  (polyline (pts (xy 74.295 15.875) (xy 74.295 72.39))
+    (stroke (width 0) (type default) (color 0 0 0 0))
+  )
+  (polyline (pts (xy 212.09 15.875) (xy 212.09 72.39))
     (stroke (width 0) (type default) (color 0 0 0 0))
   )
@@
     (effects (font (size 1.27 1.27)) (justify left bottom))
   )
+  (text "MicroSD Card Slot" (at 193.04 53.975 0)
+    (effects (font (size 1.27 1.27)) (justify left bottom))
+  )
+  (global_label "SPI1_SD_MOSI" (shape input) (at 105.41 28.575 180) (fields_autoplaced)
+    (effects (font (size 1.27 1.27)) (justify right))
+    (property "Intersheet References" "${INTERSHEET_REFS}" (id 0) (at 89.6921 28.4956 0)
+      (effects (font (size 1.27 1.27)) (justify right) hide)
+    )
+  )
+  (global_label "SPI1_SD_MISO" (shape input) (at 192.405 36.195 0) (fields_autoplaced)
+    (effects (font (size 1.27 1.27)) (justify left))
+    (property "Intersheet References" "${INTERSHEET_REFS}" (id 0) (at 208.1229 36.1156 0)
+      (effects (font (size 1.27 1.27)) (justify left) hide)
+    )
+  )
+  (global_label "SPI1_SD_CLK" (shape input) (at 105.41 38.735 180) (fields_autoplaced)
+    (effects (font (size 1.27 1.27)) (justify right))
+    (property "Intersheet References" "${INTERSHEET_REFS}" (id 0) (at 90.7202 38.6556 0)
+      (effects (font (size 1.27 1.27)) (justify right) hide)
+    )
+  )
+  (global_label "SPI1_SD_CS" (shape input) (at 105.41 23.495 180) (fields_autoplaced)
+    (effects (font (size 1.27 1.27)) (justify right))
+    (property "Intersheet References" "${INTERSHEET_REFS}" (id 0) (at 91.8088 23.4156 0)
+      (effects (font (size 1.27 1.27)) (justify right) hide)
+    )
+  )
   (symbol (lib_id "power:GND") (at 49.53 45.085 0) (unit 1)
     (in_bom yes) (on_board yes) (fields_autoplaced)
@@
       (effects (font (size 1.27 1.27)) hide)
     )
+    (pin "1")
+  )
+  (symbol (lib_id "power:GND") (at 182.245 62.23 0) (unit 1)
+    (in_bom yes) (on_board yes) (fields_autoplaced)
+    (property "Reference" "#PWR0102" (id 0) (at 182.245 68.58 0)
+      (effects (font (size 1.27 1.27)) hide)
+    )
+    (property "Value" "GND" (id 1) (at 182.245 66.675 0))
+    (property "Footprint" "" (id 2) (at 182.245 62.23 0)
+      (effects (font (size 1.27 1.27)) hide)
+    )
+    (property "Datasheet" "" (id 3) (at 182.245 62.23 0)
+      (effects (font (size 1.27 1.27)) hide)
+    )
+    (pin "1")
+  )
+  (symbol (lib_id "MicroSD:5033981892") (at 116.205 28.575 0) (unit 1)
+    (in_bom yes) (on_board yes) (fields_autoplaced)
+    (property "Reference" "J2" (id 0) (at 149.225 17.145 0)
+      (effects (font (size 1.524 1.524)))
+    )
+    (property "Value" "MicroSD" (id 1) (at 149.225 20.955 0)
+      (effects (font (size 1.524 1.524)))
+    )
+    (property "Footprint" "KiCAD Footprints:MicroSD" (id 2) (at 149.225 22.479 0)
+      (effects (font (size 1.524 1.524)) hide)
+    )
+    (property "Datasheet" "https://www.farnell.com/datasheets/2701368.pdf" (id 3) (at 116.205 28.575 0)
+      (effects (font (size 1.524 1.524)) hide)
+    )
+    (pin "1")
+    (pin "10")
+    (pin "2")
+    (pin "3")
+    (pin "4")
+    (pin "5")
+    (pin "11")
+    (pin "14")
+    (pin "12")
+    (pin "13")
+    (pin "6")
+    (pin "7")
+    (pin "8")
+    (pin "9")
+  )
+  (symbol (lib_id "power:+3V3") (at 83.82 33.655 0) (unit 1)
+    (in_bom yes) (on_board yes)
+    (property "Reference" "#PWR0101" (id 0) (at 83.82 37.465 0)
+      (effects (font (size 1.27 1.27)) hide)
+    )
+    (property "Value" "+3V3" (id 1) (at 86.995 31.75 0))
+    (property "Footprint" "" (id 2) (at 83.82 33.655 0)
+      (effects (font (size 1.27 1.27)) hide)
+    )
+    (property "Datasheet" "" (id 3) (at 83.82 33.655 0)
+      (effects (font (size 1.27 1.27)) hide)
+    )

Commit message: Updates of HW Desgin
Parts:
- added J4: USB C, KiCAD Footprints:usb_c_amphenol, symbol USB_C:12401826E412A
Connections:
- new net USB_D+: J4.A6 (D+_1)
- new net USB_D-: J4.A7 (D-_1)
Changed lines of the file:
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@@
+    (stroke (width 0) (type default) (color 0 0 0 0))
+  )
+  (wire (pts (xy 51.435 104.775) (xy 59.055 104.775))
     (stroke (width 0) (type default) (color 0 0 0 0))
   )
@@
   )
   (wire (pts (xy 159.385 56.515) (xy 159.385 59.69))
+    (stroke (width 0) (type default) (color 0 0 0 0))
+  )
+  (wire (pts (xy 41.275 102.235) (xy 59.055 102.235))
     (stroke (width 0) (type default) (color 0 0 0 0))
   )
@@
     )
   )
+  (global_label "USB_D+" (shape input) (at 41.275 102.235 180) (fields_autoplaced)
+    (effects (font (size 1.27 1.27)) (justify right))
+    (property "Intersheet References" "${INTERSHEET_REFS}" (id 0) (at 31.2419 102.1556 0)
+      (effects (font (size 1.27 1.27)) (justify right) hide)
+    )
+  )
+  (global_label "USB_D-" (shape input) (at 51.435 104.775 180) (fields_autoplaced)
+    (effects (font (size 1.27 1.27)) (justify right))
+    (property "Intersheet References" "${INTERSHEET_REFS}" (id 0) (at 41.4019 104.6956 0)
+      (effects (font (size 1.27 1.27)) (justify right) hide)
+    )
+  )
   (global_label "SPI1_SD_CS" (shape input) (at 105.41 23.495 180) (fields_autoplaced)
     (effects (font (size 1.27 1.27)) (justify right))
@@
     (pin "1")
   )
+  (symbol (lib_id "power:GND") (at 88.9 129.54 0) (unit 1)
+    (in_bom yes) (on_board yes) (fields_autoplaced)
+    (property "Reference" "#PWR018" (id 0) (at 88.9 135.89 0)
+      (effects (font (size 1.27 1.27)) hide)
+    )
+    (property "Value" "GND" (id 1) (at 88.9 134.62 0))
+    (property "Footprint" "" (id 2) (at 88.9 129.54 0)
+      (effects (font (size 1.27 1.27)) hide)
+    )
+    (property "Datasheet" "" (id 3) (at 88.9 129.54 0)
+      (effects (font (size 1.27 1.27)) hide)
+    )
+    (pin "1")
+  )
   (symbol (lib_id "power:GND") (at 182.245 62.23 0) (unit 1)
     (in_bom yes) (on_board yes) (fields_autoplaced)
@@
     (pin "1")
     (pin "10")
+    (pin "11")
+    (pin "12")
+    (pin "13")
+    (pin "14")
     (pin "2")
     (pin "3")
     (pin "4")
     (pin "5")
-    (pin "11")
-    (pin "14")
-    (pin "12")
-    (pin "13")
     (pin "6")
     (pin "7")
@@
     (pin "1")
   )
+  (symbol (lib_id "USB_C:12401826E412A") (at 59.055 89.535 0) (unit 1)
+    (in_bom yes) (on_board yes) (fields_autoplaced)
+    (property "Reference" "J4" (id 0) (at 75.565 81.915 0))
+    (property "Value" "USB C" (id 1) (at 75.565 84.455 0))
+    (property "Footprint" "KiCAD Footprints:usb_c_amphenol" (id 2) (at 88.265 86.995 0)
+      (effects (font (size 1.27 1.27)) (justify left) hide)
+    )
+    (property "Datasheet" "https://cdn.amphenol-cs.com/media/wysiwyg/files/drawing/12401826.pdf" (id 3) (at 88.265 89.535 0)
+      (effects (font (size 1.27 1.27)) (justify left) hide)
+    )
+    (property "Description" "USB-C (USB TYPE-C) USB 3.2 Gen 2 (USB 3.1 Gen 2, Superspeed + (USB 3.1)) Receptacle Connector 24 Position Surface Mount, Right Angle; Through Hole" (id 4) (at 88.265 92.075 0)
+      (effects (font (size 1.27 1.27)) (justify left) hide)
+    )
+    (property "Height" "3.43" (id 5) (at 88.265 94.615 0)
+      (effects (font (size 1.27 1.27)) (justify left) hide)
+    )
+    (property "Mouser Part Number" "523-12401826E412A" (id 6) (at 88.265 97.155 0)
+      (effects (font (size 1.27 1.27)) (justify left) hide)
+    )
+    (property "Mouser Price/Stock" "https://www.mouser.co.uk/ProductDetail/Amphenol-Commercial-Products/12401826E412A?qs=PzGy0jfpSMuVNsoRPQ3afw%3D%3D" (id 7) (at 88.265 99.695 0)
+      (effects (font (size 1.27 1.27)) (justify left) hide)
+    )
+    (property "Manufacturer_Name" "Amphenol" (id 8) (at 88.265 102.235 0)
+      (effects (font (size 1.27 1.27)) (justify left) hide)
+    )
+    (property "Manufacturer_Part_Number" "12401826E412A" (id 9) (at 88.265 104.775 0)
+      (effects (font (size 1.27 1.27)) (justify left) hide)
+    )
+    (pin "A1")
+    (pin "A10")
+    (pin "A11")
+    (pin "A12")
+    (pin "A2")
+    (pin "A3")
+    (pin "A4")
+    (pin "A5")
+    (pin "A6")
+    (pin "A7")
+    (pin "A8")
+    (pin "A9")
+    (pin "B1")
+    (pin "B10")
+    (pin "B11")
+    (pin "B12")
+    (pin "B2")
+    (pin "B3")
+    (pin "B4")
+    (pin "B5")
+    (pin "B6")
+    (pin "B7")
+    (pin "B8")
+    (pin "B9")
+    (pin "MH1")
+    (pin "MH2")
+    (pin "MH3")
+    (pin "MH4")
+  )
   (symbol (lib_id "Connector:Conn_01x02_Female") (at 38.735 42.545 180) (unit 1)
