File: HW Design/Main Board/KiCAD Files/internal_sensors.kicad_sch (KiCad schematic)
At the start: 2 parts, among them U7 BMM150, U8 BMI088

Commit message: hw desgign updates
Parts:
- added C5: 100uF, Capacitor_SMD:C_1206_3216Metric, symbol Device:C
- added C6: 10uF, Capacitor_SMD:C_1206_3216Metric, symbol Device:C
- added C7, C8: C, Capacitor_SMD:C_1206_3216Metric, symbol Device:C
- added JP1, JP2: SolderJumper_3_Bridged12, Jumper:SolderJumper-3_P1.3mm_Open_Pad1.0x1.5mm_NumberLabels, symbol Jumper:SolderJumper_3_Bridged12
- added R3, R5: R, Resistor_SMD:R_1206_3216Metric, symbol Device:R
- added R4, R6: 4k7, Resistor_SMD:R_1206_3216Metric, symbol Device:R
Connections:
- net xxx: now reaches U8.1 (INT2)
- net xxx: now also U8.12 (INT3), U8.13 (INT4), U8.16 (INT1)
- net IMU_AD2: now reaches U8.10 (SDO2)
- net IMU_AD2: now also JP2.2 (C)
- net +3V3: now reaches U8.11 (VDDIO)
- net +3V3: now also U8.14 (CSB1), U8.3 (VDD), U8.7 (PS), C5.1, C6.1, C7.1, C8.1, R3.1, R4.2, R5.1, R6.2
- net IMU_AD1: now reaches U8.15 (SDO1)
- net IMU_AD1: now also JP1.2 (C)
- net GND: now reaches U8.4 (GNDA)
- net GND: now also U8.6 (GNDIO), C5.2, C6.2, C7.2, C8.2, JP1.3 (B), JP2.3 (B)
- net I2C1_IMU_SCL: now reaches U8.8 (SCL/SCK)
- net I2C1_IMU_SDA: now reaches U8.9 (SDA/SDI)
- net I2C1_IMU_SDA: now also R3.2, R5.2
- new net: JP2.1 (A), R6.1
- new net: JP1.1 (A), R4.1
Other:
- note added: "I2C Addressing Solder Jumpers"
- note added: "IMU"
- moved on the sheet: U7, U8

Commit message: Updates of HW Desgin
Parts:
- removed C6: 10uF, Capacitor_SMD:C_1206_3216Metric, symbol Device:C
- removed C8: C, Capacitor_SMD:C_1206_3216Metric, symbol Device:C
- removed R3, R5: R, Resistor_SMD:R_1206_3216Metric, symbol Device:R
- added C27, C28: 100nF, symbol Device:C_Small
- added JP3, JP4: SolderJumper_3_Bridged12, Jumper:SolderJumper-3_P1.3mm_Open_Pad1.0x1.5mm_NumberLabels, symbol Jumper:SolderJumper_3_Bridged12
- added R10, R12: 4k7, Resistor_SMD:R_1206_3216Metric, symbol Device:R
- C5: value 100uF -> 100nF
- C7: value C -> 100nF
Connections:
- net I2C1_IMU_SCL is gone; now on net I2C1_SCL: U8.8 (SCL/SCK)
- net I2C1_IMU_SDA is gone; now on net I2C1_SDA: U8.9 (SDA/SDI)
- net +3V3: now also R4.1, R6.1, U7.A1 (PS), U7.B2 (VDDIO), U7.E5 (VDD), U8.2 (NC), C27.1, C28.1, R10.2, R12.1; no longer R4.2, R6.2
- net GND: now also JP1.1 (A), JP2.1 (A), U7.C5 (GND), U7.E1 (GND), U7.E3 (GND), C27.2, C28.2, JP3.1 (A), JP4.1 (A); no longer JP1.3 (B), JP2.3 (B)
- net I2C1_SCL: now reaches U7.A3 (SCK)
- net MAG_AD2: now reaches U7.A5 (CSB)
- net MAG_AD2: now also JP4.2 (C)
- net I2C1_SDA: now reaches U7.B4 (SDI)
- net MAG_AD1: now reaches U7.C1 (SDO)
- net MAG_AD1: now also JP3.2 (C)
- net INT_MAG: now reaches U7.D2 (INT)
- net DRY_MAG: now reaches U7.D4 (DRY)
- net IMU_AD1 renamed ACC_AD
- net IMU_AD2 renamed GYR_AD
- new net: JP4.3 (B), R12.2
- new net: JP3.3 (B), R10.1
- new net: JP2.3 (B), R6.2
- new net: JP1.3 (B), R4.2
Other:
- note added: "IMU I2C Addressing Solder Jumpers"
- note added: "Magnetometer"
- note added: "Magnetometer I2C Addressing Solder Jumpers 2xGND -> 0x10"
- note removed: "I2C Addressing Solder Jumpers"
- moved on the sheet: C5, C7, JP1, JP2, R4, R6, U7
