File: HW Design/Main Board/KiCAD Files/mcu_f4.kicad_sch (KiCad schematic)
At the start: 6 parts, among them U5 STM32F446ZETx, Y1 Crystal_GND2

Commit message: hw desgign updates
Parts:
- removed C3: 100nF, symbol Device:C
- removed C4: 1uF, symbol Device:C
- removed R1: 0, symbol Device:R
- added C? (x12): 100n, Capacitor_SMD:C_1206_3216Metric, symbol Device:C
- added C?: 4u7, Capacitor_SMD:C_1206_3216Metric, symbol Device:C
- added C? (x2): 12p, Capacitor_SMD:C_1206_3216Metric, symbol Device:C
- added C?: 1u, Capacitor_SMD:C_1206_3216Metric, symbol Device:C
- added C? (x2): 2u2, symbol Device:C_Small
- added C?: 10n, Capacitor_SMD:C_1206_3216Metric, symbol Device:C
- added L?: 39n, symbol Device:L_Small
- added R?: 10k, symbol Device:R_Small
- added SW?: SW_SPDT, symbol Switch:SW_SPDT
- R2: footprint (none) -> Resistor_SMD:R_1206_3216Metric
- U5: value STM32F446ZETx -> STM32F446ZET6
- Y1: value Crystal_GND2 -> 16MHZ
Connections:
- net RCC_OSC_IN is gone; now on net HSE_IN: U5.23 (PH0)
- net GND: now also C?.2, C?.2, C?.2, C?.2, C?.2, C?.2, C?.2, C?.2, C?.2, C?.2, C?.2, C?.2, C?.2, C?.2, C?.2, C?.2, C?.2, C?.2, C?.2, SW?.3 (C)
- net SWDIO: now reaches U5.105 (PA13)
- net at U5.106 (VCAP_2): now also C?.1
- net +3V3: now reaches U5.108 (VDD)
- net +3V3: now also U5.121 (VDD), U5.131 (VDD), U5.144 (VDD), U5.17 (VDD), U5.30 (VDD), U5.39 (VDD), U5.52 (VDD), U5.6 (VBAT), U5.62 (VDD), U5.72 (VDD), U5.84 (VDD), C?.1, C?.1, C?.1, C?.1, C?.1, C?.1, C?.1, C?.1, C?.1, C?.1, C?.1, C?.1, C?.1, L?.1
- net SWCLK: now reaches U5.109 (PA14)
- net SWO: now reaches U5.133 (PB3)
- net I2C1_IMU_SCL: now reaches U5.136 (PB6)
- net I2C1_IMU_SDA: now reaches U5.137 (PB7)
- net BOOT0: now reaches U5.143 (PDR_ON)
- net BOOT0: now also R?.1
- net CAN1_RX: now reaches U5.26 (PC0)
- net CAN1_TX: now reaches U5.27 (PC1)
- net +3.3VA: now reaches U5.33 (VDDA)
- net +3.3VA: now also C?.1, C?.1, L?.2
- net SPI1_SD_CS: now reaches U5.40 (PA4)
- net SPI1_SD_CLK: now reaches U5.41 (PA5)
- net SPI1_SD_MISO: now reaches U5.42 (PA6)
- net SPI1_SD_MOSI: now reaches U5.43 (PA7)
- net at U5.71 (VCAP_1): now also C?.1
- net HSE_IN: now reaches Y1.1
- net HSE_IN: now also C?.1; no longer R2.2
- net at Y1.3: now also R2.1, C?.1
- net F4_CAN1_RX renamed USB_D-
- net F4_CAN1_TX renamed USB_D+
- net F4_CAN2_RX: no longer names the net of U5.73 (PB12)
- net F4_CAN2_TX: no longer names the net of U5.74 (PB13)
- net RCC_OSC_OUT renamed HSE_OUT
- net HSE_OUT: now also R2.2; no longer R2.1
- new net: R?.2, SW?.2 (B)
Other:
- note added: "Load Cap = 2 * (Load Cap Osc - Cstray) Cstrat: est 5-6 pF Load Cap Osc - see datasheet Check Feed Resistor value"
- note added: "Low ESR Caps"
- note added: "MCU Power Filtering"
- note added: "Main MCU analog power line filtering"
- note added: "Main MCU power line decoupling 1*4u7 BulkCapacitor + 1 100n Decoupling Capacitor per VBAT & VDD"
- note removed: "Calculate Caps"
- moved on the sheet: R2, Y1

Commit message: Updates of HW Desgin
Parts:
- removed C? (x2): 2u2, symbol Device:C_Small
- removed U5: STM32F446ZET6, Package_QFP:LQFP-144_20x20mm_P0.5mm, symbol MCU_ST_STM32F4:STM32F446ZETx
- added C4: 2u2, symbol Device:C_Small
- added U5: STM32F446RETx, Package_QFP:LQFP-64_10x10mm_P0.5mm, symbol MCU_ST_STM32F4:STM32F446RETx
- gave numbers to parts that had none: 20
Connections:
- net +3.3VA: now also U5.13 (VDDA)
- net +3V3: now also U5.1 (VBAT), U5.19 (VDD), U5.32 (VDD), U5.48 (VDD), U5.64 (VDD)
- net CAN1_RX: now also U5.8 (PC0)
- net CAN1_TX: now also U5.9 (PC1)
- net GND: now also C4.2, U5.12 (VSSA), U5.18 (VSS), U5.31 (VSS), U5.47 (VSS), U5.63 (VSS)
- net HSE_IN: now also U5.5 (PH0)
- net HSE_OUT: now also U5.6 (PH1)
- net NRST: now also U5.7 (NRST)
- net SPI1_SD_CLK: now also U5.21 (PA5)
- net SPI1_SD_CS: now also U5.20 (PA4)
- net SPI1_SD_MISO: now also U5.22 (PA6)
- net SPI1_SD_MOSI: now also U5.23 (PA7)
- net SWCLK: now also U5.49 (PA14)
- net SWDIO: now also U5.46 (PA13)
- net SWO: now also U5.55 (PB3)
- net USB_D+: now also U5.45 (PA12)
- net USB_D-: now also U5.44 (PA11)
- new net: C4.1, U5.30 (VCAP_1)
- new net I2C1_SCL: U5.58 (PB6)
- new net I2C1_SDA: U5.59 (PB7)
