File: HW Design/Main Board/KiCAD Files/power_managment.kicad_sch (KiCad schematic)
At the start: 3 parts, among them U1 LM3940IMP-3.3/NOPB

Commit message: hw desgign updates
Parts:
- removed C1: 0.47 uF, symbol Device:C
- removed C2: 33uF, symbol Device:C
- removed U1: LM3940IMP-3.3/NOPB, Package_TO_SOT_SMD:SOT-223, symbol LM3940:LM3940IMP-3.3/NOPB
- added C? (x2): 10n, symbol Device:C
- added C?: 10u, symbol Device:C
- added D?: D_Schottky, symbol Device:D_Schottky
- added F?: 1A, symbol Device:Polyfuse
- added FB?: 600 @ 600MHz, symbol Device:FerriteBead
- added L?: L, symbol Device:L
- added Q?: AO3401A, Package_TO_SOT_SMD:SOT-23, symbol Transistor_FET:AO3401A
- added R?: 68k, symbol Device:R
- added R?: 100k, symbol Device:R
- added U?: MP2359, symbol New_Library:MP2359
Connections:
- net GND: now also C?.2, D?.2 (A), Q?.1 (G), R?.2, U?.2 (GND)
- new net: C?.1, L?.2
- new net: FB?.1, Q?.2 (S)
- new net: F?.1, Q?.3 (D)
- new net +12V: F?.2
- new net BUCK_BST: C?.1, U?.1 (BST)
- new net BUCK_EN: R?.1, R?.2, U?.4 (EN)
- new net BUCK_FB: U?.3 (FB)
- new net BUCK_IN: C?.1, FB?.2, R?.1, U?.5 (IN)
- new net BUCK_SW: C?.2, D?.1 (K), L?.1, U?.6 (SW)
Other:
- note removed: "33uF is minimum, check if bigger is needed ESR limits are <0.1; 1> ohm (<1 ohm for <200mA)"

Commit message: Updates of HW Desgin
Parts:
- gave numbers to parts that had none: 11
Changed lines of the file:
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@@
   (symbol (lib_id "power:GND") (at 160.02 99.06 0) (unit 1)
     (in_bom yes) (on_board yes) (fields_autoplaced)
-    (property "Reference" "#PWR?" (id 0) (at 160.02 105.41 0)
+    (property "Reference" "#PWR032" (id 0) (at 160.02 105.41 0)
       (effects (font (size 1.27 1.27)) hide)
     )
@@
   (symbol (lib_id "Device:D_Schottky") (at 160.02 90.17 270) (unit 1)
     (in_bom yes) (on_board yes) (fields_autoplaced)
-    (property "Reference" "D?" (id 0) (at 162.56 88.5824 90)
+    (property "Reference" "D1" (id 0) (at 162.56 88.5824 90)
       (effects (font (size 1.27 1.27)) (justify left))
     )
@@
   (symbol (lib_id "power:GND") (at 82.55 91.44 0) (unit 1)
     (in_bom yes) (on_board yes) (fields_autoplaced)
-    (property "Reference" "#PWR?" (id 0) (at 82.55 97.79 0)
+    (property "Reference" "#PWR023" (id 0) (at 82.55 97.79 0)
       (effects (font (size 1.27 1.27)) hide)
     )
@@
   (symbol (lib_id "power:GND") (at 82.55 41.91 0) (unit 1)
     (in_bom yes) (on_board yes) (fields_autoplaced)
-    (property "Reference" "#PWR?" (id 0) (at 82.55 48.26 0)
+    (property "Reference" "#PWR05" (id 0) (at 82.55 48.26 0)
       (effects (font (size 1.27 1.27)) hide)
     )
@@
   (symbol (lib_id "Device:C") (at 187.96 90.17 0) (unit 1)
     (in_bom yes) (on_board yes) (fields_autoplaced)
-    (property "Reference" "C?" (id 0) (at 191.77 88.8999 0)
+    (property "Reference" "C3" (id 0) (at 191.77 88.8999 0)
       (effects (font (size 1.27 1.27)) (justify left))
     )
@@
   (symbol (lib_id "power:GND") (at 124.46 60.96 0) (unit 1)
     (in_bom yes) (on_board yes) (fields_autoplaced)
-    (property "Reference" "#PWR?" (id 0) (at 124.46 67.31 0)
+    (property "Reference" "#PWR031" (id 0) (at 124.46 67.31 0)
       (effects (font (size 1.27 1.27)) hide)
     )
@@
   (symbol (lib_id "power:GND") (at 50.8 41.91 0) (unit 1)
     (in_bom yes) (on_board yes) (fields_autoplaced)
-    (property "Reference" "#PWR?" (id 0) (at 50.8 48.26 0)
+    (property "Reference" "#PWR04" (id 0) (at 50.8 48.26 0)
       (effects (font (size 1.27 1.27)) hide)
     )
@@
   (symbol (lib_id "Device:R") (at 124.46 53.34 0) (unit 1)
     (in_bom yes) (on_board yes) (fields_autoplaced)
-    (property "Reference" "R?" (id 0) (at 127 52.0699 0)
+    (property "Reference" "R7" (id 0) (at 127 52.0699 0)
       (effects (font (size 1.27 1.27)) (justify left))
     )
@@
   (symbol (lib_id "Device:C") (at 82.55 35.56 0) (unit 1)
     (in_bom yes) (on_board yes) (fields_autoplaced)
-    (property "Reference" "C?" (id 0) (at 86.36 34.2899 0)
+    (property "Reference" "C1" (id 0) (at 86.36 34.2899 0)
       (effects (font (size 1.27 1.27)) (justify left))
     )
@@
   (symbol (lib_id "Transistor_FET:AO3401A") (at 50.8 33.02 90) (unit 1)
     (in_bom yes) (on_board yes) (fields_autoplaced)
-    (property "Reference" "Q?" (id 0) (at 50.8 22.86 90))
+    (property "Reference" "Q1" (id 0) (at 50.8 22.86 90))
     (property "Value" "AO3401A" (id 1) (at 50.8 25.4 90))
     (property "Footprint" "Package_TO_SOT_SMD:SOT-23" (id 2) (at 52.705 27.94 0)
@@
   (symbol (lib_id "New_Library:MP2359") (at 82.55 82.55 0) (unit 1)
     (in_bom yes) (on_board yes) (fields_autoplaced)
-    (property "Reference" "U?" (id 0) (at 82.55 64.77 0))
+    (property "Reference" "U1" (id 0) (at 82.55 64.77 0))
     (property "Value" "MP2359" (id 1) (at 83.82 67.31 0))
     (property "Footprint" "" (id 2) (at 80.01 82.804 0)
@@
   (symbol (lib_id "Device:Polyfuse") (at 34.29 30.48 270) (unit 1)
     (in_bom yes) (on_board yes)
-    (property "Reference" "F?" (id 0) (at 34.29 27.94 90))
+    (property "Reference" "F1" (id 0) (at 34.29 27.94 90))
     (property "Value" "1A" (id 1) (at 34.29 33.02 90))
     (property "Footprint" "" (id 2) (at 29.21 31.75 0)
@@
   (symbol (lib_id "Device:C") (at 132.08 86.36 0) (unit 1)
     (in_bom yes) (on_board yes) (fields_autoplaced)
-    (property "Reference" "C?" (id 0) (at 135.89 85.0899 0)
+    (property "Reference" "C2" (id 0) (at 135.89 85.0899 0)
       (effects (font (size 1.27 1.27)) (justify left))
     )
@@
   (symbol (lib_id "Device:L") (at 176.53 81.28 90) (unit 1)
     (in_bom yes) (on_board yes) (fields_autoplaced)
-    (property "Reference" "L?" (id 0) (at 176.53 74.93 90))
+    (property "Reference" "L1" (id 0) (at 176.53 74.93 90))
     (property "Value" "L" (id 1) (at 176.53 77.47 90))
     (property "Footprint" "" (id 2) (at 176.53 81.28 0)
@@
   (symbol (lib_id "Device:FerriteBead") (at 69.85 30.48 90) (unit 1)
     (in_bom yes) (on_board yes) (fields_autoplaced)
-    (property "Reference" "FB?" (id 0) (at 69.7992 22.86 90))
+    (property "Reference" "FB1" (id 0) (at 69.7992 22.86 90))
     (property "Value" "600 @ 600MHz" (id 1) (at 69.7992 25.4 90))
     (property "Footprint" "" (id 2) (at 69.85 32.258 90)
@@
   (symbol (lib_id "power:+12V") (at 21.59 27.94 0) (unit 1)
     (in_bom yes) (on_board yes) (fields_autoplaced)
-    (property "Reference" "#PWR?" (id 0) (at 21.59 31.75 0)
+    (property "Reference" "#PWR03" (id 0) (at 21.59 31.75 0)
       (effects (font (size 1.27 1.27)) hide)
     )
@@
   (symbol (lib_id "Device:R") (at 124.46 38.1 0) (unit 1)
     (in_bom yes) (on_board yes) (fields_autoplaced)
-    (property "Reference" "R?" (id 0) (at 127 36.8299 0)
-      (effects (font (size 1.27 1.27)) (justify left))
-    )
+    (property "Reference" "R1" (id 0) (at 127 36.8299 0)
+      (effects (font (size 1.27 1.27)) (justify left))
+    )
